File: Hardware/Spindle.kicad_sch (KiCad schematic)
At the start: 14 parts, among them J1 USB_C_Receptacle_USB2.0_16P, U1 ESP32-S3, U2 BQ24074RGT, U3 MCP1700x-330xxTT

Commit message: Updated schematic
Parts:
- removed C1: 10n, symbol Device:C
- removed C2, C7: 1u, symbol Device:C
- removed C3, C5, C6: 0.1u, symbol Device:C
- removed C4: 10u, symbol Device:C
- removed D1: ESD9B3.3ST5G, Diode_SMD:D_SOD-923, symbol Diode:ESD9B3.3ST5G
- removed U1: ESP32-S3, Package_DFN_QFN:QFN-56-1EP_7x7mm_P0.4mm_EP4x4mm, symbol MCU_Espressif:ESP32-S3
- added C10, C11: 12p, symbol Device:C
- added C8: 1u, symbol Device:C
- added C9: 4.7u, symbol Device:C
- added D2, D3: LED, symbol Device:LED
- added J2: Conn_01x02_Pin, symbol Connector:Conn_01x02_Pin
- added J3: Conn_01x24_Pin, symbol Connector:Conn_01x24_Pin
- added J4: Micro_SD_Card, symbol Connector:Micro_SD_Card
- added R3: 46.4K, symbol Device:R
- added R4: 1.18K, symbol Device:R
- added R5: 1.13K, symbol Device:R
- added R6, R7: 1.5K, symbol Device:R
- added TH1: Thermistor, symbol Device:Thermistor
- added U1: RP2350A, Package_DFN_QFN:QFN-60-1EP_7x7mm_P0.4mm_EP3.4x3.4mm, symbol MCU_RaspberryPi:RP2350A
- added Y1: 12mhz, symbol Device:Crystal_GND23
Connections:
- net +3V3: now also J4.4 (VDD)
- net GND: now also U2.17 (VSS), U2.8 (VSS), C10.2, C11.2, C8.2, C9.2, J4.6 (VSS), J4.SH (SHIELD), R3.2, R4.2, R5.2, Y1.2 (G), Y1.3 (G)
- net USB_D+: now also U1.52 (USB_DP)
- net USB_D-: now also U1.51 (USB_DM)
- net VBUS: now also U2.13 (IN), C8.1
- net TS: now reaches U2.1 (TS)
- net TS: now also TH1.1
- net OUT: now reaches U2.10 (OUT), U2.11 (OUT)
- net OUT: now also C9.1, R6.1, R7.1
- net at U2.12 (ILIM): now also R4.1
- net TMR: now reaches U2.14 (TMR)
- net at U2.15 (ITERM): now also R3.1
- net at U2.16 (ISET): now also R5.1
- net BAT: now reaches U2.2 (BAT), U2.3 (BAT)
- net BAT: now also J2.1 (Pin_1)
- net CE: now reaches U2.4 (~{CE})
- net EN2: now reaches U2.5 (EN2)
- net EN1: now reaches U2.6 (EN1)
- net PGOOD: now reaches U2.7 (~{PGOOD})
- net PGOOD: now also D3.1 (K)
- net CHG: now reaches U2.9 (~{CHG})
- net CHG: now also D2.1 (K)
- new net: D2.2 (A), R6.2
- new net: D3.2 (A), R7.2
- new net: J2.2 (Pin_2), TH1.2
- new net: U1.1 (IOVDD), U1.11 (IOVDD), U1.20 (IOVDD), U1.30 (IOVDD), U1.38 (IOVDD), U1.45 (IOVDD)
- new net: U1.23 (DVDD), U1.39 (DVDD), U1.6 (DVDD)
- new net BS1: J3.8 (Pin_8)
- new net BUSY: J3.9 (Pin_9)
- new net CS#: J3.12 (Pin_12)
- new net D/C#: J3.11 (Pin_11)
- new net GDR: J3.2 (Pin_2)
- new net RES#: J3.10 (Pin_10)
- new net RESE: J3.3 (Pin_3)
- new net SCL: J3.13 (Pin_13)
- new net SDA: J3.14 (Pin_14)
- new net SD_CLK: J4.5 (CLK), U1.4 (GPIO2)
- new net SD_CMD: J4.3 (CMD), U1.5 (GPIO3)
- new net SD_DAT0: J4.7 (DAT0), U1.2 (GPIO0)
- new net SD_DAT3: J4.2 (DAT3/CD), U1.3 (GPIO1)
- new net TSCL: J3.6 (Pin_6)
- new net TSDA: J3.7 (Pin_7)
- new net VCI: J3.16 (Pin_16)
- new net VCOM: J3.24 (Pin_24)
- new net VDD: J3.18 (Pin_18)
- new net VDDIO: J3.15 (Pin_15)
- new net VGH: J3.21 (Pin_21)
- new net VGL: J3.23 (Pin_23)
- new net VPP: J3.19 (Pin_19)
- new net VSH1: J3.20 (Pin_20)
- new net VSH2: J3.5 (Pin_5)
- new net VSL: J3.22 (Pin_22)
- new net VSS: J3.17 (Pin_17)
- new net XIN: C10.1, U1.21 (XIN), Y1.1
- new net XOUT: C11.1, U1.22 (XOUT), Y1.4
- no-connect marks 0 -> 4
Other:
- note added: "Crystal"
- note added: "E-Ink Display connector"
- note added: "Micro-SD Reader"
- note added: "RP2350a"
- note removed: "Capacitors"
- note removed: "ESP32-S3"
- moved on the sheet: J1, R1, R2, U2, U3

Commit message: updated schematic
Parts:
- removed C10, C11: 12p, symbol Device:C
- removed D3: LED, symbol Device:LED
- removed R1, R2: 5.1K, symbol Device:R
- removed R3: 46.4K, symbol Device:R
- removed R4: 1.18K, symbol Device:R
- removed R5: 1.13K, symbol Device:R
- removed R6, R7: 1.5K, symbol Device:R
- removed TH1: Thermistor, symbol Device:Thermistor
- added C1, C2: 15p, symbol Device:C
- added C3, C4, C5, C6, C7: 1u, symbol Device:C
- added D1: GREEN, symbol Device:LED
- added D3, D4: D_Schottky, symbol Device:D_Schottky
- added L1: 10u, symbol Device:L
- added Q1: BSS138, symbol Transistor_FET:Q_NMOS_GSD
- added R1: 60.4K, symbol Device:R_US
- added R2: 10K, symbol Device:R_US
- added R3, R4, R7: 1.5K, symbol Device:R_US
- added R5, R6: 5.1K, symbol Device:R_US
- added R8: 1K, symbol Device:R_US
- added R9: 0.47, symbol Device:R_US
- C9: value 4.7u -> 1u
- D2: value LED -> RED
Connections:
- net CE is gone; now on net GND: U2.4 (~{CE})
- net EN1 is gone; now on net GND: U2.6 (EN1)
- net EN2 is gone; now on net +3V3: U2.5 (EN2)
- net RESE is gone; now on net TP_SCL: J3.3 (Pin_3)
- net SCL is gone; now on net GND: J3.13 (Pin_13)
- net SDA is gone; now on net +3V3: J3.14 (Pin_14)
- net TSCL is gone; now on net TP_RST: J3.6 (Pin_6)
- net TSDA is gone; now on net EPD_BUSY: J3.7 (Pin_7)
- net VCI is gone; now on net GND: J3.16 (Pin_16)
- net VDD is gone; now on net +3V3: J3.18 (Pin_18)
- net VDDIO is gone; now on net +3V3: J3.15 (Pin_15)
- net VSH2 is gone; now on net TP_INT: J3.5 (Pin_5)
- net +3V3: now also J3.2 (Pin_2), L1.1
- net CS#: now also U1.13 (GPIO9); no longer J3.12 (Pin_12)
- net D/C#: now also U1.12 (GPIO8); no longer J3.11 (Pin_11)
- net GDR: now also L1.2, Q1.1 (G), Q1.3 (D); no longer J3.2 (Pin_2)
- net GND: now also J2.1 (Pin_1), J3.1 (Pin_1), C1.1, C2.2, C3.2, C4.2, C5.2, C6.2, C7.2, R1.2, R2.2, R5.2, R6.1, R7.1, R8.2; no longer C8.2, C9.2
- net PGOOD: now also D1.1 (K)
- net RES#: now also U1.16 (GPIO12); no longer J3.10 (Pin_10)
- net VBUS: no longer C8.1, U3.3 (VI)
- net at U2.16 (ISET): now also R8.1
- net at D2.2 (A): now also R3.1
- net at J1.A5 (CC1): now also R5.1
- net at J1.B5 (CC2): now also R6.2
- net at U2.12 (ILIM): now also R7.2
- net BAT+: now reaches J2.2 (Pin_2)
- net BAT+: now also U2.2 (BAT), U2.3 (BAT)
- net ESD_SCLK: now reaches U1.14 (GPIO10)
- net ESD_SDIN: now reaches U1.15 (GPIO11)
- net EPD_BUSY: now reaches U1.17 (GPIO13)
- net TP_SDA: now reaches U1.18 (GPIO14)
- net TP_SDA: now also J3.4 (Pin_4)
- net TP_SCL: now reaches U1.19 (GPIO15)
- net TP_INT: now reaches U1.27 (GPIO16)
- net TP_RST: now reaches U1.28 (GPIO17)
- removed net BAT: J2.1 (Pin_1), U2.2 (BAT), U2.3 (BAT)
- net BS1 renamed EPD_RST
- net BUSY renamed EPD_DC
- net OUT renamed BQ_OUT
- net BQ_OUT: now also U3.3 (VI), R3.2, R4.2; no longer C9.1
- net TMR renamed BQ_TMR
- net BQ_TMR: now also R1.1
- net TS: no longer names the net of U2.1 (TS)
- net TS: now also R2.1
- net USB_D+ renamed DATA+
- net DATA+: no longer U1.52 (USB_DP)
- net USB_D- renamed DATA-
- net DATA-: no longer U1.51 (USB_DM)
- net VCOM renamed EPD_PIN24
- net VGH renamed EPD_PIN21
- net EPD_PIN21: now also C6.1
- net VGL renamed EPD_PIN23
- net VPP renamed EPD_PIN19
- net EPD_PIN19: now also C4.1
- net VSH1 renamed EPD_PIN20
- net EPD_PIN20: now also C5.1
- net VSL renamed EPD_PIN22
- net EPD_PIN22: now also C7.1
- net VSS renamed EPD_PIN17
- net EPD_PIN17: now also C3.1
- net XIN: no longer names the net of Y1.1
- net XIN: now also C2.1; no longer U1.21 (XIN)
- net XOUT: no longer names the net of Y1.4
- net XOUT: now also C1.2; no longer U1.22 (XOUT)
- new net: D1.2 (A), R4.1
- new net EPD_CS: J3.10 (Pin_10)
- new net EPD_SCLK: J3.11 (Pin_11)
- new net EPD_SDIP: J3.12 (Pin_12)
Other:
- note added: "ALL CAPACITORS SHOULD BE OF 25V"
- note added: "E-Ink Display Boost circuit"
- moved on the sheet: J3, U2, U3

Commit message: worked on the schematic
Parts:
- removed C6, C7, C8, C9: 1u, symbol Device:C
- removed D3, D4: D_Schottky, symbol Device:D_Schottky
- removed Q1: BSS138, symbol Transistor_FET:Q_NMOS_GSD
- removed R9: 0.47, symbol Device:R_US
- added C10, C11, C12, C6, C7, C8, C9: 1u, symbol Device:C_Small
- added D3, D4, D5: MBR0530, Diode_SMD:D_SOD-123, symbol Diode:MBR0530
- added Q1: Si1308EDL, Package_TO_SOT_SMD:SOT-323_SC-70, symbol Transistor_FET:Si1308EDL
- added R10: 1M, symbol Device:R_Small
- added R9: 2.2R, symbol Device:R_Small
- C3, C5: value 1u -> 4.7u
- L1: value 10u -> 47u
Connections:
- net CS# is gone; now on net EPD_CS: U1.13 (GPIO9)
- net EPD_DC is gone; now on net EPD_BUSY: J3.9 (Pin_9)
- net EPD_PIN21 is gone; now on net VGH: J3.21 (Pin_21)
- net EPD_SCLK is gone; now on net EPD_D/C#: J3.11 (Pin_11)
- net EPD_SDIP is gone; now on net EPD_CS: J3.12 (Pin_12)
- net RES# is gone; now on net EPD_RST: U1.16 (GPIO12)
- net +3V3: now also C5.1; no longer J3.14 (Pin_14), J3.15 (Pin_15), J3.18 (Pin_18), J3.2 (Pin_2)
- net EPD_BUSY: no longer J3.7 (Pin_7)
- net EPD_CS: no longer J3.10 (Pin_10)
- net EPD_RST: now also J3.10 (Pin_10); no longer J3.8 (Pin_8)
- net GDR: now also J3.2 (Pin_2), Q1.1 (G), R10.1; no longer L1.2
- net GND: now also J3.17 (Pin_17), J3.8 (Pin_8), C10.2, C11.2, C12.2, C6.2, C7.2, C8.2, C9.2, D4.1 (K), R10.2, R9.2; no longer C3.2, J3.1 (Pin_1), J3.13 (Pin_13), J3.16 (Pin_16)
- net TP_SCL: now also J3.6 (Pin_6); no longer J3.3 (Pin_3)
- net TP_SDA: now also J3.7 (Pin_7); no longer J3.4 (Pin_4)
- net D/C# renamed EPD_D/C#
- net EPD_PIN17: no longer names the net of C3.1
- net EPD_PIN17: now also D3.1 (K), D4.2 (A); no longer J3.17 (Pin_17)
- net EPD_PIN19 renamed VGH
- net VGH: now also D5.1 (K); no longer J3.19 (Pin_19)
- net EPD_PIN20 renamed VSH1
- net VSH1: now also C9.1; no longer C5.1
- net EPD_PIN22 renamed VSL
- net VSL: now also C10.1
- net EPD_PIN23 renamed VGL
- net VGL: now also C11.1, D3.2 (A)
- net EPD_PIN24 renamed VCOM
- net VCOM: now also C12.1
- net ESD_SCLK renamed EPD_SCK
- net EPD_SCK: now also J3.13 (Pin_13)
- net ESD_SDIN renamed EPD_SDI
- net EPD_SDI: now also J3.14 (Pin_14)
- net TP_INT: no longer names the net of J3.5 (Pin_5)
- net TP_INT: now also C6.1; no longer U1.27 (GPIO16)
- net TP_RST: no longer names the net of U1.28 (GPIO17)
- net TP_RST: no longer J3.6 (Pin_6)
- new net: C3.2, Q1.3 (D)
- new net: D5.2 (A), L1.2
- new net RESE: J3.3 (Pin_3), Q1.2 (S), R9.1
- new net VDD: C8.1, J3.18 (Pin_18)
- new net VDDIO: C7.1, J3.15 (Pin_15), J3.16 (Pin_16)
- new net VPP: J3.19 (Pin_19)
- no-connect marks 4 -> 6
Other:
- note added: "E-Ink Display connector and boost circuit"
- note removed: "E-Ink Display Boost circuit"
- note removed: "E-Ink Display connector"
- moved on the sheet: J3

Commit message: updated schematic
Parts:
- added C13, C14, C15, C16, C17, C18, C19, C20, C21, C24: 100n, Capacitor_SMD:C_0402_1005Metric, symbol Device:C
- added C23, C25, C26: 4.7u, Capacitor_SMD:C_0402_1005Metric, symbol Device:C
- added R11: 10K, Resistor_SMD:R_0402_1005Metric, symbol Device:R_Small
- added SW1: SW_Push, Button_Switch_SMD:SW_SPST_PTS810, symbol Switch:SW_Push
- C1, C10, C11, C12, C2, C3, C4, C5, C6, C7, C8, C9: footprint (none) -> Capacitor_SMD:C_0402_1005Metric
- D1, D2: footprint (none) -> LED_SMD:LED_0402_1005Metric
- J1: footprint (none) -> Connector_USB:USB_C_Receptacle_HCTL_HC-TYPE-C-16P-01A
- J2: footprint (none) -> Connector_PinHeader_2.54mm:PinHeader_1x02_P2.54mm_Vertical
- J3: footprint (none) -> Connector_FFC-FPC:Hirose_FH12-24S-0.5SH_1x24-1MP_P0.50mm_Horizontal
- J4: footprint (none) -> Connector_Card:microSD_HC_Molex_104031-0811
- L1: footprint (none) -> Inductor_SMD:L_10.4x10.4_H4.8
- R1, R10, R2, R3, R4, R5, R6, R7, R8, R9: footprint (none) -> Resistor_SMD:R_0402_1005Metric
- Y1: footprint (none) -> Crystal:Crystal_SMD_3225-4Pin_3.2x2.5mm
Connections:
- net +3V3: now also U1.1 (IOVDD), U1.11 (IOVDD), U1.20 (IOVDD), U1.30 (IOVDD), U1.38 (IOVDD), U1.44 (ADC_AVDD), U1.45 (IOVDD), U1.46 (VREG_AVDD), U1.49 (VREG_VIN), U1.53 (USB_OTP_VDD), U1.54 (QSPI_IOVDD), C13.1, C14.1, C15.1, C16.1, C17.1, C18.1, C19.1, C20.1, C21.1, C25.1, C26.1, R11.1
- net DATA+: now also U1.52 (USB_DP)
- net DATA-: now also U1.51 (USB_DM)
- net GND: now also U1.47 (VREG_PGND), U1.61 (GND), C13.2, C14.2, C15.2, C16.2, C17.2, C18.2, C19.2, C20.2, C21.2, C23.2, C24.2, C25.2, C26.2, SW1.1
- net XOUT: now reaches C2.1, Y1.1
- net XOUT: now also U1.22 (XOUT)
- net XIN: now reaches C1.2, Y1.4
- net XIN: now also U1.21 (XIN)
- net DVDD: now reaches U1.23 (DVDD), U1.39 (DVDD), U1.6 (DVDD)
- net DVDD: now also C23.1, C24.1
- net RUN: now reaches U1.26 (RUN)
- net RUN: now also R11.2, SW1.2
- net VREG_VX: now reaches U1.48 (VREG_LX)
- net VREG_FB: now reaches U1.50 (VREG_FB)

Commit message: Started PCB layout
Parts:
- added C27: 4.7u, Capacitor_SMD:C_0402_1005Metric, symbol Device:C
- added L2: 3.3u, Inductor_SMD:L_Sunlord_SWPA5040S, symbol Device:L
Connections:
- net GND: now also C27.2
- net VREG_FB renamed +1V1
- net +1V1: now also C27.1, L2.2
- net VREG_VX: no longer names the net of U1.48 (VREG_LX)
- net VREG_VX: now also L2.1
Other:
- moved on the sheet: C13, C14, C15, C16, C17, C18

Commit message: updated PCB
Parts:
- added U4: W25Q128JVP, Package_SON:WSON-8-1EP_6x5mm_P1.27mm_EP3.4x4.3mm, symbol Memory_Flash:W25Q128JVP
Connections:
- net +3V3: now also U4.8 (VCC)
- net GND: now also U4.4 (GND), U4.9 (EP)
- net FLASH_IO3: now reaches U1.55 (QSPI_SD3)
- net FLASH_IO3: now also U4.7 (~{HOLD}/~{RESET}/IO_{3})
- net FLASH_CLK: now reaches U1.56 (QSPI_SCLK)
- net FLASH_CLK: now also U4.6 (CLK)
- net FLASH_IO0: now reaches U1.57 (QSPI_SD0)
- net FLASH_IO0: now also U4.5 (DI/IO_{0})
- net FLASH_IO2: now reaches U1.58 (QSPI_SD2)
- net FLASH_IO2: now also U4.3 (~{WP}/IO_{2})
- net FLASH_IO1: now reaches U1.59 (QSPI_SD1)
- net FLASH_IO1: now also U4.2 (DO/IO_{1})
- net FLASH_CS: now reaches U1.60 (~{QSPI_SS})
- net FLASH_CS: now also U4.1 (~{CS})
- no-connect marks 6 -> 26
Other:
- note added: "Flash"

Commit message: Completed PCB
Parts:
- added R12, R13, R14, R15, R16: 10K, Resistor_SMD:R_0402_1005Metric, symbol Device:R_Small
- added SW2, SW3, SW4, SW5, SW6: SW_Push, Button_Switch_SMD:SW_SPST_PTS810, symbol Switch:SW_Push
- L1: footprint Inductor_SMD:L_10.4x10.4_H4.8 -> Inductor_THT:L_Radial_D6.0mm_P4.00mm
Connections:
- net +3V3: now also R12.1, R13.1, R14.1, R15.1, R16.1
- net GND: now also SW2.1, SW3.1, SW4.1, SW5.1, SW6.1
- net SW_UP: now reaches U1.31 (GPIO19)
- net SW_UP: now also R12.2, SW2.2
- net SW_DOWN: now reaches U1.32 (GPIO20)
- net SW_DOWN: now also R15.2, SW5.2
- net SW_CENTRE: now reaches U1.33 (GPIO21)
- net SW_CENTRE: now also R14.2, SW4.2
- net SW_RIGHT: now reaches U1.34 (GPIO22)
- net SW_RIGHT: now also R16.2, SW6.2
- net SW_LEFT: now reaches U1.35 (GPIO23)
- net SW_LEFT: now also R13.2, SW3.2
- no-connect marks 26 -> 21

Commit message: Updated CAD
Parts:
- added H1, H2: MountingHole, MountingHole:MountingHole_3.2mm_M3, symbol Mechanical:MountingHole
- added R17: 10K, Resistor_SMD:R_0402_1005Metric, symbol Device:R_Small
- added R18: 470, Resistor_SMD:R_0402_1005Metric, symbol Device:R_Small
- added U5: <value>, RP_RM2:rpi_rmc20452t, symbol RPI_RMC20452T:RPI_RMC20452T
Connections:
- net +3V3: now also U5.14 (VDDIO), U5.16 (VIN)
- net GND: now also U5.1 (GND), U5.11 (GND), U5.15 (GND), U5.21 (GND), U5.4 (GND), U5.7 (GND)
- net GPIO24: now reaches U1.36 (GPIO24)
- net GPIO24: now also R17.1, R18.2, U5.5 (DI)
- net GPIO25: now reaches U1.37 (GPIO25)
- net GPIO25: now also U5.9 (CS)
- net RM_SCLK: now reaches U1.43 (GPIO29/ADC3)
- net RM_SCLK: now also U5.3 (SCLK)
- net GPIO5: now reaches U1.8 (GPIO5)
- net GPIO5: now also U5.12 (WL_ON), U5.13 (BT_ON)
- new net: R17.2, U5.10 (nIRQ)
- new net: R18.1, U5.6 (DO)
- no-connect marks 21 -> 20
Other:
- note added: "Radio Mudule"
