File: Hardware/Spindle.kicad_sch (KiCad schematic)
At the start: 70 parts, among them J1 USB_C_Receptacle_USB2.0_16P, J2 Conn_01x02_Pin, J3 Conn_01x24_Pin, J4 Micro_SD_Card, Q1 Si1308EDL, SW1 SW_Push, SW2 SW_Push, SW3 SW_Push, SW4 SW_Push, SW5 SW_Push, SW6 SW_Push, U1 RP2350A, U2 BQ24074RGT, U3 MCP1700x-330xxTT, U4 W25Q128JVP, U5 <value>, Y1 12mhz

Commit message: better routing
Parts:
- removed R12, R13, R14, R15, R16: 10K, Resistor_SMD:R_0402_1005Metric, symbol Device:R_Small
- removed Y1: 12mhz, Crystal:Crystal_SMD_3225-4Pin_3.2x2.5mm, symbol Device:Crystal_GND23
- added R19: 10K, Resistor_SMD:R_0402_1005Metric, symbol Device:R_Small
- added SW7: SW_Push, Button_Switch_SMD:SW_SPST_PTS810, symbol Switch:SW_Push
- added Y1: Crystal_GND24, Crystal:Crystal_SMD_3225-4Pin_3.2x2.5mm, symbol Device:Crystal_GND24
- C23: value 4.7u -> 100n
- L1: footprint Inductor_THT:L_Radial_D6.0mm_P4.00mm -> Inductor_SMD:L_Sunlord_SWPA5040S
- L2: footprint Inductor_SMD:L_Sunlord_SWPA5040S -> easyeda2kicad:IND-SMD_L2.0-W1.6_AOTA-B201610S3R3-101-T
Connections:
- net DVDD is gone; now on net +1V1: C23.1, C24.1, U1.23 (DVDD), U1.39 (DVDD), U1.6 (DVDD)
- net SW_CENTRE is gone; now on net +3V3: SW4.2, U1.33 (GPIO21)
- net SW_DOWN is gone; now on net +3V3: SW5.2, U1.32 (GPIO20)
- net SW_RIGHT is gone; now on net +3V3: SW6.2, U1.34 (GPIO22)
- net +3V3: now also R11.2, SW2.2, SW3.2, U1.10 (GPIO7), U1.42 (GPIO28/ADC2), R19.2; no longer R11.1
- net FLASH_CS: now also R19.1, SW7.2
- net GND: now also R2.1, SW7.1, Y1.2 (G), Y1.4 (G); no longer R2.2
- net RUN: now also R11.1; no longer R11.2
- net XIN: now also Y1.1
- net XOUT: now also Y1.3
- net at C3.2, Q1.3 (D): now also D5.2 (A), L1.2
- net at U2.1 (TS): now also R2.2; no longer R2.1
- net SW_LEFT: no longer names the net of U1.35 (GPIO23)
- net SW_LEFT: no longer SW3.2
- net SW_UP: no longer names the net of U1.31 (GPIO19)
- net SW_UP: no longer SW2.2
- no-connect marks 20 -> 23
Other:
- note added: "3v3 LDO regulator"
- note added: "RP2350A"
- note removed: "3v3 converter"
- note removed: "Crystal"
- note removed: "RP2350a"
- moved on the sheet: C13, C14, C15, C16, C17, C18, C19, C20, C21, C23, C24, C25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

Commit message: did CAD
Parts:
- added R12: 1K, Resistor_SMD:R_0402_1005Metric, symbol Device:R_US
Connections:
- net +3V3: no longer SW2.2, SW3.2, SW4.2, SW5.2, SW6.2, U1.10 (GPIO7), U1.32 (GPIO20), U1.33 (GPIO21), U1.34 (GPIO22), U1.42 (GPIO28/ADC2)
- net GND: now also R12.2; no longer J1.SH (SHIELD)
- net at U2.15 (ITERM): now also R12.1
- new net SW_CENTRE: SW3.2, U1.33 (GPIO21)
- new net SW_DOWN: SW6.2, U1.32 (GPIO20)
- new net SW_LEFT: SW2.2, U1.10 (GPIO7)
- new net SW_RIGHT: SW4.2, U1.34 (GPIO22)
- new net SW_UP: SW5.2, U1.42 (GPIO28/ADC2)
- no-connect marks 23 -> 24
