File: Hardware/Spindle.kicad_pcb (KiCad board)
At the start: 2 copper layers, 37 parts, among them J1 USB_C_Receptacle_USB2.0_16P, J2 Conn_01x02_Pin, J3 Conn_01x24_Pin, J4 Micro_SD_Card, Q1 Si1308EDL, U1 RP2350A, U2 BQ24074RGT, U3 MCP1700x-330xxTT, Y1 12mhz

Commit message: Started PCB layout
Parts:
- added C13: 100n, Capacitor_SMD:C_0402_1005Metric, F.Cu at (486.4, 89.3)
- added C14: 100n, Capacitor_SMD:C_0402_1005Metric, F.Cu at (486.4, 91.3)
- added C15: 100n, Capacitor_SMD:C_0402_1005Metric, F.Cu at (489.3, 79.5)
- added C16: 100n, Capacitor_SMD:C_0402_1005Metric, F.Cu at (489.3, 81.4)
- added C17: 100n, Capacitor_SMD:C_0402_1005Metric, F.Cu at (489.3, 83.4)
- added C18: 100n, Capacitor_SMD:C_0402_1005Metric, F.Cu at (489.3, 85.4)
- added C19: 100n, Capacitor_SMD:C_0402_1005Metric, F.Cu at (489.3, 87.3)
- added C20: 100n, Capacitor_SMD:C_0402_1005Metric, F.Cu at (489.3, 89.3)
- added C21: 100n, Capacitor_SMD:C_0402_1005Metric, F.Cu at (489.3, 91.3)
- added C23: 4.7u, Capacitor_SMD:C_0402_1005Metric, F.Cu at (492.2, 79.5)
- added C24: 100n, Capacitor_SMD:C_0402_1005Metric, F.Cu at (492.2, 81.4)
- added C25: 4.7u, Capacitor_SMD:C_0402_1005Metric, F.Cu at (492.2, 83.4)
- added C26: 4.7u, Capacitor_SMD:C_0402_1005Metric, F.Cu at (492.2, 85.4)
- added C27: 4.7u, Capacitor_SMD:C_0402_1005Metric, F.Cu at (492.2, 87.3)
- added L2: 3.3u, Inductor_SMD:L_Sunlord_SWPA5040S, F.Cu at (496.6, 72.8)
- added R11: 10K, Resistor_SMD:R_0402_1005Metric, F.Cu at (486.5, 101.2)
- added SW1: SW_Push, Button_Switch_SMD:SW_SPST_PTS810, F.Cu at (489.9, 71.9)
- moved Q1 194.0 mm to (501.9, 76.5)
- moved U2 182.7 mm to (503.0, 72.2)
- moved Y1 177.5 mm to (502.3, 104.6)
- moved L1 176.7 mm to (499.9, 84.4)
- moved D1 174.2 mm to (494.5, 103.4)
- moved D2 174.2 mm to (494.5, 105.4)
- moved D4 166.7 mm to (502.6, 97.3)
- moved U3 161.9 mm to (490.4, 104.6)
- moved C8 156.9 mm to (486.4, 79.5)
- moved C1 154.5 mm to (483.6, 79.5)
- moved C2 154.5 mm to (483.6, 81.4)
- moved C3 154.5 mm to (483.6, 83.4)
- moved C4 154.5 mm to (483.6, 85.4)
- moved C11 151.1 mm to (486.4, 85.4)
- moved C5 148.9 mm to (483.6, 87.3)
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Connections:
- net Net-(U1-DVDD-Pad23) renamed /DVDD
- C1 pad 2: Net-(C1-Pad2) -> /XIN
- C2 pad 1: Net-(C2-Pad1) -> /XOUT
- U1 pad 1: Net-(U1-IOVDD-Pad1) -> +3V3
- U1 pad 11: Net-(U1-IOVDD-Pad1) -> +3V3
- U1 pad 20: Net-(U1-IOVDD-Pad1) -> +3V3
- U1 pad 21: unconnected-(U1-XIN-Pad21) -> /XIN
- U1 pad 22: unconnected-(U1-XOUT-Pad22) -> /XOUT
- U1 pad 26: unconnected-(U1-RUN-Pad26) -> /RUN
- U1 pad 30: Net-(U1-IOVDD-Pad1) -> +3V3
- U1 pad 38: Net-(U1-IOVDD-Pad1) -> +3V3
- U1 pad 44: unconnected-(U1-ADC_AVDD-Pad44) -> +3V3
- U1 pad 45: Net-(U1-IOVDD-Pad1) -> +3V3
- U1 pad 46: unconnected-(U1-VREG_AVDD-Pad46) -> +3V3
- U1 pad 47: unconnected-(U1-VREG_PGND-Pad47) -> GND
- U1 pad 48: unconnected-(U1-VREG_LX-Pad48) -> Net-(U1-VREG_LX)
- U1 pad 49: unconnected-(U1-VREG_VIN-Pad49) -> +3V3
- U1 pad 50: unconnected-(U1-VREG_FB-Pad50) -> +1V1
- U1 pad 51: unconnected-(U1-USB_DM-Pad51) -> /DATA-
- U1 pad 52: unconnected-(U1-USB_DP-Pad52) -> /DATA+
- U1 pad 53: unconnected-(U1-USB_OTP_VDD-Pad53) -> +3V3
- U1 pad 54: unconnected-(U1-QSPI_IOVDD-Pad54) -> +3V3
- U1 pad 61: unconnected-(U1-GND-Pad61) -> GND
- Y1 pad 1: Net-(C2-Pad1) -> /XOUT
- Y1 pad 4: Net-(C1-Pad2) -> /XIN
Other:
- board outline added: 50 x 40 mm

Commit message: updated PCB
Parts:
- removed R2: 10K, Resistor_SMD:R_0402_1005Metric
- added U4: W25Q128JVP, Package_SON:WSON-8-1EP_6x5mm_P1.27mm_EP3.4x4.3mm, F.Cu at (450.2, 162.1)
- moved SW1 109.6 mm to (456.1, 176.1), turned to 180 degrees
- moved U2 104.8 mm to (436.6, 153.3), turned to 180 degrees
- moved L2 98.6 mm to (455.9, 162.6), turned to 180 degrees
- moved Y1 89.3 mm to (449.1, 176.4), turned to 180 degrees
- moved C27 81.1 mm to (454.7, 159.3)
- moved C9 78.9 mm to (450.1, 98.0), turned to 0 degrees
- moved Q1 75.0 mm to (442.6, 122.5)
- moved C10 73.7 mm to (450.1, 100.0), turned to 0 degrees
- moved C12 66.5 mm to (450.1, 103.9), turned to 0 degrees
- moved J2 65.1 mm to (441.5, 151.1)
- moved D3 60.0 mm to (466.2, 110.5)
- moved D5 56.6 mm to (466.2, 117.2)
- moved D1 54.2 mm to (442.3, 117.8)
- moved D2 54.2 mm to (442.3, 119.8)
- moved U3 48.3 mm to (443.1, 114.6)
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Connections:
- U1 pad 55: unconnected-(U1-QSPI_SD3-Pad55) -> /FLASH_IO3
- U1 pad 56: unconnected-(U1-QSPI_SCLK-Pad56) -> /FLASH_CLK
- U1 pad 57: unconnected-(U1-QSPI_SD0-Pad57) -> /FLASH_IO0
- U1 pad 58: unconnected-(U1-QSPI_SD2-Pad58) -> /FLASH_IO2
- U1 pad 59: unconnected-(U1-QSPI_SD1-Pad59) -> /FLASH_IO1
- U1 pad 60: unconnected-(U1-~{QSPI_SS}-Pad60) -> /FLASH_CS
Routing:
- net /FLASH_IO1: track 0.00 -> 12.9 mm, vias 0 -> 2
- net /FLASH_CS: track 0.00 -> 12.5 mm, vias 0 -> 2
- net +1V1: track 0.00 -> 11.2 mm, vias 0 -> 2
- net /FLASH_IO2: track 0.00 -> 9.94 mm, vias 0 -> 2
- net +3V3: track 0.00 -> 7.90 mm
- net /RUN: track 0.00 -> 7.15 mm
- net Net-(U1-VREG_LX): track 0.00 -> 6.81 mm
- net /XIN: track 0.00 -> 4.71 mm
- net /BAT+: track 0.00 -> 3.91 mm
- net /XOUT: track 0.00 -> 2.35 mm
- net /FLASH_IO0: track 0.00 -> 1.91 mm
- net /FLASH_IO3: track 0.00 -> 1.89 mm
- net /FLASH_CLK: track 0.00 -> 1.55 mm
- added copper zone on In2.Cu, net +3V3
- added copper zone on B.Cu, net GND
- added copper zone on F.Cu, net GND
- added copper zone on In1.Cu, net GND
Other:
- copper layers 2 -> 4

Commit message: Completed PCB
Parts:
- added R12: 10K, Resistor_SMD:R_0402_1005Metric, B.Cu at (447.6, 172.6)
- added R13: 10K, Resistor_SMD:R_0402_1005Metric, B.Cu at (440.8, 177.3)
- added R14: 10K, Resistor_SMD:R_0402_1005Metric, B.Cu at (447.6, 177.3)
- added R15: 10K, Resistor_SMD:R_0402_1005Metric, B.Cu at (447.6, 182.0)
- added R16: 10K, Resistor_SMD:R_0402_1005Metric, B.Cu at (454.3, 177.3)
- added R2: 10K, Resistor_SMD:R_0402_1005Metric, F.Cu at (432.3, 161.3)
- added SW2: SW_Push, Button_Switch_SMD:SW_SPST_PTS810, B.Cu at (446.0, 170.2)
- added SW3: SW_Push, Button_Switch_SMD:SW_SPST_PTS810, B.Cu at (439.2, 175.0)
- added SW4: SW_Push, Button_Switch_SMD:SW_SPST_PTS810, B.Cu at (446.0, 175.0)
- added SW5: SW_Push, Button_Switch_SMD:SW_SPST_PTS810, B.Cu at (446.0, 179.7)
- added SW6: SW_Push, Button_Switch_SMD:SW_SPST_PTS810, B.Cu at (452.7, 175.0)
- L1: footprint Inductor_SMD:L_10.4x10.4_H4.8 -> Inductor_THT:L_Radial_D6.0mm_P4.00mm
- moved C8 83.7 mm to (446.4, 179.7), turned to 90 degrees
- moved C9 81.7 mm to (447.3, 179.7), turned to 90 degrees
- moved L1 81.2 mm to (459.8, 182.2), turned to 180 degrees
- moved C10 79.7 mm to (448.8, 179.7), turned to 90 degrees
- moved C11 79.3 mm to (426.8, 177.7), turned to 180 degrees
- moved C3 78.7 mm to (436.9, 177.9)
- moved C4 77.8 mm to (450.6, 179.7), turned to -90 degrees
- moved D3 76.3 mm to (430.2, 177.7), turned to 180 degrees
- moved C12 75.8 mm to (449.7, 179.7), turned to 90 degrees
- moved D4 75.3 mm to (430.2, 180.0)
- moved C23 74.9 mm to (443.0, 169.8), turned to 180 degrees
- moved C6 73.7 mm to (440.1, 179.2), turned to 90 degrees
- moved C15 73.2 mm to (441.9, 168.4), turned to -90 degrees
- moved C7 71.8 mm to (445.4, 179.7), turned to 90 degrees
- moved C16 71.4 mm to (441.0, 168.4), turned to -90 degrees
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Connections:
- J3 pad : GND -> (no net)
- J4 pad : GND -> (no net)
- U1 pad 31: unconnected-(U1-GPIO19-Pad31) -> /SW_UP
- U1 pad 32: unconnected-(U1-GPIO20-Pad32) -> /SW_DOWN
- U1 pad 33: unconnected-(U1-GPIO21-Pad33) -> /SW_CENTRE
- U1 pad 34: unconnected-(U1-GPIO22-Pad34) -> /SW_RIGHT
- U1 pad 35: unconnected-(U1-GPIO23-Pad35) -> /SW_LEFT
Routing:
- net +3V3: track 7.90 -> 59.6 mm, vias 0 -> 19
- net /SW_DOWN: track 0.00 -> 38.5 mm, vias 0 -> 2
- net /SW_LEFT: track 0.00 -> 38.2 mm, vias 0 -> 2
- net GND: track 0.00 -> 30.1 mm, vias 0 -> 17
- net /SW_CENTRE: track 0.00 -> 29.2 mm, vias 0 -> 1
- net /SW_RIGHT: track 0.00 -> 27.7 mm, vias 0 -> 2
- net /DATA-: track 0.00 -> 26.1 mm, vias 0 -> 2
- net /VGL: track 0.00 -> 25.3 mm, vias 0 -> 2
- net /TP_SDA: track 0.00 -> 24.4 mm, vias 0 -> 2
- net /SD_CLK: track 0.00 -> 23.6 mm, vias 0 -> 2
- net /TP_SCL: track 0.00 -> 23.3 mm, vias 0 -> 2
- net /DVDD: track 0.00 -> 22.7 mm, vias 0 -> 4
- net /DATA+: track 0.00 -> 22.4 mm, vias 0 -> 2
- net /SW_UP: track 0.00 -> 22.3 mm, vias 0 -> 1
- net /EPD_RST: track 0.00 -> 22.1 mm, vias 0 -> 2
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- added copper zone on In1.Cu, net +3V3
- added copper zone on In2.Cu, net GND
- removed copper zone on In1.Cu, net GND
Other:
- board size 50 x 40 mm -> 40 x 40 mm
- board text added: "Charging"
- board text added: "Full Charge"

Commit message: Updated CAD
Parts:
- added H1: MountingHole, MountingHole:MountingHole_3.2mm_M3, F.Cu at (427.9, 184.3)
- added H2: MountingHole, MountingHole:MountingHole_3.2mm_M3, F.Cu at (459.4, 152.0)
- added R17: 10K, Resistor_SMD:R_0402_1005Metric, B.Cu at (451.4, 171.8)
- added R18: 470, Resistor_SMD:R_0402_1005Metric, B.Cu at (456.5, 173.9)
- added U5: <value>, RP_RM2:rpi_rmc20452t, B.Cu at (460.2, 165.1)
- moved C24 4.02 mm to (443.1, 170.7), turned to 180 degrees
- moved D4 2.01 mm to (432.2, 180.2)
- moved J4 0.15 mm to (457.0, 162.3), turned to -90 degrees
Connections:
- U1 pad 36: unconnected-(U1-GPIO24-Pad36) -> /GPIO24
- U1 pad 37: unconnected-(U1-GPIO25-Pad37) -> /GPIO25
- U1 pad 43: unconnected-(U1-GPIO29/ADC3-Pad43) -> /RM_SCLK
- U1 pad 8: unconnected-(U1-GPIO5-Pad8) -> /GPIO5
Routing:
- net /RM_SCLK: track 0.00 -> 31.0 mm, vias 0 -> 2
- net /GPIO24: track 0.00 -> 29.3 mm, vias 0 -> 2
- net /GPIO25: track 0.00 -> 16.6 mm, vias 0 -> 2
- net /GPIO5: track 0.00 -> 13.0 mm, vias 0 -> 2
- net /SD_DAT0: track 16.8 -> 28.5 mm, vias 2 -> 3
- net /SD_DAT3: track 21.3 -> 31.5 mm
- net /SD_CMD: track 17.0 -> 27.1 mm
- net /SD_CLK: track 23.6 -> 33.1 mm
- net /SW_UP: track 22.3 -> 30.9 mm, vias 1 -> 4
- net Net-(U5-nIRQ): track 0.00 -> 6.62 mm
- net +3V3: track 59.6 -> 64.6 mm, vias 19 -> 22
- net Net-(U5-DO): track 0.00 -> 2.29 mm
- net /SW_LEFT: track 38.2 -> 39.3 mm
- net Net-(D3-K): track 7.06 -> 8.05 mm
- net /DVDD: track 22.7 -> 21.9 mm
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
Commit message: better routing
Parts:
- removed R12, R13, R14, R15, R16: 10K, Resistor_SMD:R_0402_1005Metric
- added R19: 10K, Resistor_SMD:R_0402_1005Metric, F.Cu at (440.7, 154.5)
- added SW7: SW_Push, Button_Switch_SMD:SW_SPST_PTS810, F.Cu at (436.9, 153.4)
- C23: value 4.7u -> 100n
- J4: moved to B.Cu
- L1: footprint Inductor_THT:L_Radial_D6.0mm_P4.00mm -> Inductor_SMD:L_Sunlord_SWPA5040S
- L2: footprint Inductor_SMD:L_Sunlord_SWPA5040S -> easyeda2kicad:IND-SMD_L2.0-W1.6_AOTA-B201610S3R3-101-T
- R17, R18, U5: moved to F.Cu
- Y1: value 12mhz -> Crystal_GND24
- moved SW1 32.9 mm to (456.7, 184.4)
- moved R11 32.2 mm to (460.6, 185.4)
- moved L1 31.6 mm to (429.1, 174.7), turned to 0 degrees
- moved D1 29.0 mm to (456.6, 156.1), turned to 90 degrees
- moved R3 28.8 mm to (454.5, 158.9), turned to -90 degrees
- moved J1 28.8 mm to (447.8, 150.7), turned to 180 degrees
- moved R4 28.1 mm to (453.5, 158.9), turned to -90 degrees
- moved D2 27.9 mm to (455.7, 156.1), turned to 90 degrees
- moved R8 27.8 mm to (459.1, 163.7)
- moved R2 27.8 mm to (460.1, 162.9), turned to 90 degrees
- moved R1 26.8 mm to (457.5, 163.7)
- moved J2 26.7 mm to (461.8, 157.2)
- moved U2 26.7 mm to (457.7, 160.0)
- moved J4 26.6 mm to (430.5, 159.8)
- moved R7 26.3 mm to (455.4, 162.1), turned to 90 degrees
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Connections:
- C23 pad 1: /DVDD -> +1V1
- C24 pad 1: /DVDD -> +1V1
- C3 pad 2: Net-(Q1-D) -> Net-(D5-A)
- Q1 pad 3: Net-(Q1-D) -> Net-(D5-A)
- R11 pad 1: +3V3 -> /RUN
- R11 pad 2: /RUN -> +3V3
- R2 pad 1: Net-(U2-TS) -> GND
- R2 pad 2: GND -> Net-(U2-TS)
- SW2 pad 2: /SW_UP -> /SW_LEFT
- SW3 pad 2: /SW_LEFT -> /SW_CENTRE
- SW4 pad 2: /SW_CENTRE -> /SW_RIGHT
- SW5 pad 2: /SW_DOWN -> /SW_UP
- SW6 pad 2: /SW_RIGHT -> /SW_DOWN
- U1 pad 10: unconnected-(U1-GPIO7-Pad10) -> /SW_LEFT
- U1 pad 23: /DVDD -> +1V1
- U1 pad 31: /SW_UP -> unconnected-(U1-GPIO19-Pad31)
- U1 pad 35: /SW_LEFT -> unconnected-(U1-GPIO23-Pad35)
- U1 pad 39: /DVDD -> +1V1
- U1 pad 42: unconnected-(U1-GPIO28/ADC2-Pad42) -> /SW_UP
- U1 pad 6: /DVDD -> +1V1
- Y1 pad 1: /XOUT -> /XIN
- Y1 pad 3: GND -> /XOUT
- Y1 pad 4: /XIN -> GND
Routing:
- net /SW_LEFT: track 39.3 -> 8.48 mm, vias 2 -> 1
- net +3V3: track 64.6 -> 38.7 mm, vias 22 -> 15
- net /SW_UP: track 30.9 -> 6.97 mm, vias 4 -> 1
- net /SW_DOWN: track 38.2 -> 14.6 mm, vias 2 -> 1
- net /SW_RIGHT: track 28.4 -> 6.46 mm, vias 2 -> 1
- net /DVDD: track 21.9 -> 0.00 mm, vias 4 -> 0
- net /SW_CENTRE: track 29.1 -> 7.33 mm
- net /RM_SCLK: track 31.0 -> 13.3 mm
- net /FLASH_CS: track 6.16 -> 20.4 mm, vias 2 -> 0
- net GND: track 29.7 -> 16.1 mm, vias 17 -> 30
- net /DATA-: track 26.1 -> 13.0 mm, vias 2 -> 0
- net /GPIO25: track 16.6 -> 4.01 mm, vias 2 -> 0
- net +1V1: track 19.4 -> 7.29 mm, vias 3 -> 4
- net Net-(D5-A): track 12.0 -> 0.00 mm
- net /VGH: track 6.99 -> 18.6 mm, vias 0 -> 2
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- added copper zone on F.Cu, net +1V1
- added copper zone on In2.Cu, net +1V1
- added copper zone on F.Cu, net +3V3
- added copper zone on F.Cu, net /BAT+
- added copper zone on F.Cu, net /BQ_OUT
- added copper zone on In1.Cu, net GND
- added copper zone on F.Cu, net Net-(D3-K)
- added copper zone on F.Cu, net Net-(D5-A)
- added copper zone on F.Cu, net Net-(U1-VREG_LX)
- added copper zone on F.Cu, net VBUS
- added copper zone on In2.Cu, net VBUS
- removed copper zone on In1.Cu, net +3V3
- removed copper zone on In2.Cu, net GND
Other:
- board text removed: "Charging"
- board text removed: "Full Charge"
