File: Hardware/Spindle.kicad_pcb (KiCad board)
At the start: 4 copper layers, 40 x 40 mm, 67 parts, among them J1 USB_C_Receptacle_USB2.0_16P, J2 Conn_01x02_Pin, J3 Conn_01x24_Pin, J4 Micro_SD_Card, Q1 Si1308EDL, SW1 SW_Push, SW2 SW_Push, SW3 SW_Push, SW4 SW_Push, SW5 SW_Push, SW6 SW_Push, SW7 SW_Push, U1 RP2350A, U2 BQ24074RGT, U3 MCP1700x-330xxTT, U4 W25Q128JVP, U5 <value>, Y1 Crystal_GND24

Commit message: did CAD
Parts:
- moved R5 0.34 mm to (449.1, 156.9)
Connections:
- J1 pad SH: GND -> unconnected-(J1-SHIELD-PadSH)_2
Routing:
- net GND: track 16.1 -> 9.03 mm, vias 30 -> 60
- net /SW_DOWN: track 14.6 -> 17.2 mm
- net /DATA-: track 13.0 -> 14.0 mm
- net /SD_CLK: track 22.4 -> 23.4 mm
- net /SD_CMD: track 22.4 -> 23.4 mm
- net /SD_DAT0: track 22.4 -> 23.4 mm
- net /SD_DAT3: track 22.4 -> 23.4 mm
- net /VGL: track 31.9 -> 31.2 mm
- net VBUS: track 8.38 -> 8.39 mm, vias 3 -> 5
- added copper zone on In2.Cu, net /BAT+
