File: Hardware/Spindle.kicad_pcb (KiCad board)
At the start: 4 copper layers, 40 x 40 mm, 70 parts, among them J1 USB_C_Receptacle_USB2.0_16P, J2 Conn_01x02_Pin, J3 Conn_01x24_Pin, J4 Micro_SD_Card, Q1 Si1308EDL, SW1 SW_Push, SW2 SW_Push, SW3 SW_Push, SW4 SW_Push, SW5 SW_Push, SW6 SW_Push, U1 RP2350A, U2 BQ24074RGT, U3 MCP1700x-330xxTT, U4 W25Q128JVP, U5 <value>, Y1 12mhz

Commit message: idk why
Connections:
- J3 pad : (no net) -> GND
Routing:
- net Net-(D5-A): track 12.0 -> 10.9 mm
Changed lines of the file:
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@@
 			(size 1.8 2.2)
 			(layers "F.Cu" "F.Mask" "F.Paste")
+			(net "GND")
 		)
 		(pad "" smd rect
@@
 			(size 1.8 2.2)
 			(layers "F.Cu" "F.Mask" "F.Paste")
+			(net "GND")
 		)
 		(pad "1" smd rect
@@
 	)
 	(segment
-		(start 450.3275 176.6875)
-		(end 450.3275 174.6875)
-		(width 0.2)
-		(layer "F.Cu")
-		(net "Net-(D5-A)")
-	)
-	(segment
 		(start 455.82 182.18)
-		(end 450.3275 176.6875)
+		(end 448.3275 174.6875)
 		(width 0.2)
 		(layer "F.Cu")
@@
 	)
 	(segment
-		(start 448.06 174.6875)
-		(end 450.3275 174.6875)
+		(start 448.3275 174.6875)
+		(end 448.06 174.6875)
 		(width 0.2)
 		(layer "F.Cu")
@@
 		(layers "F.Cu" "B.Cu" "In2.Cu")
 		(hatch edge 0.5)
-		(connect_pads thru_hole_only
+		(connect_pads yes
 			(clearance 0.5)
 		)
